Commit message: Last version

File: Project/Simulation/puzzlebot_description/urdf/base.xacro (robot description, xacro)
@@ -6,5 +6,5 @@
       <origin xyz="0 0 0" rpy="0 0 0"/>
       <geometry>
-        <mesh filename="package://puzzlebot_description/meshes/bases/Puzzlebot_Jetson_Lidar_Edition_Base.stl" scale="${mesh_scale} ${mesh_scale} ${mesh_scale}"/>
+        <mesh filename="package://puzzlebot_description/meshes/Puzzlebot_Jetson_Lidar_Edition_Base.stl" scale="${mesh_scale} ${mesh_scale} ${mesh_scale}"/>
       </geometry>
       <material name="yellow">

File: Project/Simulation/puzzlebot_description/urdf/puzzlebot.xacro (robot description, xacro)
@@ -1,8 +1,4 @@
 <?xml version="1.0"?>
 <robot name="puzzlebot" xmlns:xacro="http://www.ros.org/wiki/xacro">
-  <!-- ============================================================
-       PROPERTIES — Puzzlebot escalado al 70% para caber en pasillos estrechos
-       Tamano efectivo: 12.6 x 10.5 cm (era 18 x 15 cm)
-       ============================================================ -->
   <xacro:property name="mesh_scale"      value="0.7"/>
   <xacro:property name="base_mass"       value="0.5"/>
@@ -19,7 +15,5 @@
   <xacro:property name="lidar_radius"    value="0.025"/>
   <xacro:property name="lidar_height"    value="0.03"/>
-  <!-- ============================================================
-       INCLUDES — modulos del robot
-       ============================================================ -->
+  <!-- INCLUDES -->
   <xacro:include filename="$(find puzzlebot_description)/urdf/inertias.xacro"/>
   <xacro:include filename="$(find puzzlebot_description)/urdf/base.xacro"/>

File: Project/Simulation/puzzlebot_description/urdf/wheels.xacro (robot description, xacro)
@@ -6,5 +6,5 @@
         <origin xyz="0 0 0" rpy="1.5708 0 0"/>
         <geometry>
-          <mesh filename="package://puzzlebot_description/meshes/wheels/Puzzlebot_Wheel.stl" scale="${mesh_scale} ${mesh_scale} ${mesh_scale}"/>
+          <mesh filename="package://puzzlebot_description/meshes/Puzzlebot_Wheel.stl" scale="${mesh_scale} ${mesh_scale} ${mesh_scale}"/>
         </geometry>
         <material name="dark_grey">
@@ -34,5 +34,5 @@
       <origin xyz="0 0 0" rpy="0 0 0"/>
       <geometry>
-        <mesh filename="package://puzzlebot_description/meshes/wheels/Puzzlebot_Caster_Wheel.stl" scale="${mesh_scale} ${mesh_scale} ${mesh_scale}"/>
+        <mesh filename="package://puzzlebot_description/meshes/Puzzlebot_Caster_Wheel.stl" scale="${mesh_scale} ${mesh_scale} ${mesh_scale}"/>
       </geometry>
       <material name="grey">
